File: ortho-40percent.kicad_pcb (KiCad board)
At the start: 2 copper layers, 229 x 81 mm, 128 parts, among them J1 USB-C_Receptacle-24, SW1 SW_NO_4-Pin, SW10 CherryMX, SW11 CherryMX, SW12 CherryMX, SW13 CherryMX, SW14 CherryMX, SW15 CherryMX, SW16 CherryMX, SW17 CherryMX, SW18 CherryMX, SW19 CherryMX, SW2 CherryMX, SW20 CherryMX, SW21 CherryMX, SW22 CherryMX, SW23 CherryMX, SW24 CherryMX, SW25 CherryMX, SW26 CherryMX, SW27 CherryMX, SW28 CherryMX, SW29 CherryMX, SW3 CherryMX, SW30 CherryMX, SW31 CherryMX, SW32 CherryMX, SW33 CherryMX, SW34 CherryMX, SW35 CherryMX, SW36 CherryMX, SW37 CherryMX, SW38 CherryMX, SW39 CherryMX, SW4 CherryMX, SW40 CherryMX, SW41 CherryMX, SW42 CherryMX, SW43 CherryMX, SW44 CherryMX, SW45 CherryMX, SW46 CherryMX, SW47 CherryMX, SW48 CherryMX, SW49 CherryMX, SW5 CherryMX, SW50 CherryMX, SW51 CherryMX, SW6 CherryMX, SW7 CherryMX, SW8 CherryMX, SW9 CherryMX, U1 U_TPD4E05U06DQAR, U2 U_ATmega32u4-MU, Y1 XTAL_4Lead

Commit message: more routing
more routing
Connections:
- D35 pad K: /KeyMatrix/ROW5 -> /KeyMatrix/ROW3
- D47 pad K: /KeyMatrix/ROW5 -> /KeyMatrix/ROW2
- SW36 pad 1: /KeyMatrix/COL0 -> /KeyMatrix/COL10
- SW48 pad 1: /KeyMatrix/COL3 -> /KeyMatrix/COL10
Routing:
- net /KeyMatrix/COL9: track 119.2 -> 159.8 mm
- net /KeyMatrix/COL10: track 19.4 -> 43.9 mm, vias 2 -> 3
Changed lines of the file:
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@@
     (thickness 1.6)
     (drawings 71)
-    (tracks 723)
+    (tracks 736)
     (zones 0)
     (modules 128)
@@
       (net 43 "Net-(D35-PadA)"))
     (pad K smd roundrect (at -1.575 0 270) (size 0.9 0.95) (layers F.Cu F.Paste F.Mask) (roundrect_rratio 0.25)
-      (net 13 /KeyMatrix/ROW5))
+      (net 9 /KeyMatrix/ROW3))
     (model ${KIPRJMOD}/ortho-40percent.3dshapes/SOD-123.step
       (at (xyz 0 0 0))
@@
       (net 55 "Net-(D47-PadA)"))
     (pad K smd roundrect (at -1.575 0 270) (size 0.9 0.95) (layers F.Cu F.Paste F.Mask) (roundrect_rratio 0.25)
-      (net 13 /KeyMatrix/ROW5))
+      (net 8 /KeyMatrix/ROW2))
     (model ${KIPRJMOD}/ortho-40percent.3dshapes/SOD-123.step
       (at (xyz 0 0 0))
@@
       (net 43 "Net-(D35-PadA)"))
     (pad 1 smd roundrect (at 0 3.55) (size 2.55 2.5) (layers F.Cu F.Paste F.Mask) (roundrect_rratio 0.25)
-      (net 69 /KeyMatrix/COL0))
+      (net 110 /KeyMatrix/COL10))
     (pad "" np_thru_hole circle (at 5.08 -7.62 90) (size 1.7 1.7) (drill 1.7) (layers *.Cu *.Mask))
     (pad "" np_thru_hole circle (at 5.08 2.54 90) (size 1.7 1.7) (drill 1.7) (layers *.Cu *.Mask))
@@
       (net 55 "Net-(D47-PadA)"))
     (pad 1 smd roundrect (at 0 3.55) (size 2.55 2.5) (layers F.Cu F.Paste F.Mask) (roundrect_rratio 0.25)
-      (net 72 /KeyMatrix/COL3))
+      (net 110 /KeyMatrix/COL10))
     (pad "" np_thru_hole circle (at 5.08 -7.62 90) (size 1.7 1.7) (drill 1.7) (layers *.Cu *.Mask))
     (pad "" np_thru_hole circle (at 5.08 2.54 90) (size 1.7 1.7) (drill 1.7) (layers *.Cu *.Mask))
@@
   (segment (start 195.96 223.345) (end 196.635 223.345) (width 0.25) (layer F.Cu) (net 11))
   (segment (start 196.635 223.345) (end 196.71 223.42) (width 0.25) (layer F.Cu) (net 11))
+  (segment (start 118.6 227.855) (end 118.6 232.46) (width 0.25) (layer F.Cu) (net 12))
+  (segment (start 119.96 226.495) (end 118.6 227.855) (width 0.25) (layer F.Cu) (net 12))
   (segment (start 251.785 185.345) (end 252.96 185.345) (width 0.25) (layer F.Cu) (net 13))
   (segment (start 251.46 185.67) (end 251.785 185.345) (width 0.25) (layer F.Cu) (net 13))
@@
   (segment (start 252.885 166.42) (end 252.96 166.345) (width 0.25) (layer F.Cu) (net 13))
   (segment (start 251.71 166.42) (end 252.885 166.42) (width 0.25) (layer F.Cu) (net 13))
-  (segment (start 118.6 227.855) (end 118.6 232.46) (width 0.25) (layer F.Cu) (net 12))
-  (segment (start 119.96 226.495) (end 118.6 227.855) (width 0.25) (layer F.Cu) (net 12))
   (via (at 252.96 203.17) (size 0.8) (drill 0.4) (layers F.Cu B.Cu) (net 13))
   (segment (start 252.96 203.17) (end 252.96 204.345) (width 0.25) (layer F.Cu) (net 13))
@@
   (segment (start 224.72 194.67) (end 227.05 197) (width 0.25) (layer F.Cu) (net 109))
   (segment (start 222.46 194.67) (end 224.72 194.67) (width 0.25) (layer F.Cu) (net 109))
+  (segment (start 259.96 232.92) (end 262.97 232.92) (width 0.25) (layer F.Cu) (net 109))
+  (segment (start 262.97 232.92) (end 265.05 235) (width 0.25) (layer F.Cu) (net 109))
+  (segment (start 229.21 234.92) (end 239.21 234.92) (width 0.25) (layer F.Cu) (net 109))
+  (segment (start 242.46 231.67) (end 247.46 231.67) (width 0.25) (layer F.Cu) (net 109))
+  (segment (start 247.46 231.67) (end 251.21 235.42) (width 0.25) (layer F.Cu) (net 109))
+  (segment (start 239.21 234.92) (end 242.46 231.67) (width 0.25) (layer F.Cu) (net 109))
+  (segment (start 251.21 235.42) (end 257.46 235.42) (width 0.25) (layer F.Cu) (net 109))
+  (segment (start 257.46 235.42) (end 259.96 232.92) (width 0.25) (layer F.Cu) (net 109))
   (via (at 245.71 218.17) (size 0.8) (drill 0.4) (layers F.Cu B.Cu) (net 110))
   (segment (start 246.05 216) (end 246.05 217.83) (width 0.25) (layer F.Cu) (net 110))
@@
   (segment (start 246.21 234.84) (end 246.05 235) (width 0.25) (layer F.Cu) (net 110))
   (segment (start 246.21 232.92) (end 246.21 234.84) (width 0.25) (layer F.Cu) (net 110))
+  (via (at 248.21 196.92) (size 0.8) (drill 0.4) (layers F.Cu B.Cu) (net 110))
+  (segment (start 246.05 197) (end 248.13 197) (width 0.25) (layer F.Cu) (net 110))
+  (segment (start 248.13 197) (end 248.21 196.92) (width 0.25) (layer F.Cu) (net 110))
+  (segment (start 248.21 215.67) (end 245.71 218.17) (width 0.25) (layer B.Cu) (net 110))
+  (segment (start 248.21 196.92) (end 248.21 215.67) (width 0.25) (layer B.Cu) (net 110))
   (zone (net 2) (net_name GND) (layer F.Cu) (hatch edge 0.508)
     (connect_pads (clearance 0.2))

Commit message: More routing
even more routing
Connections:
- D35 pad K: /KeyMatrix/ROW3 -> /KeyMatrix/ROW2
- D47 pad K: /KeyMatrix/ROW2 -> /KeyMatrix/ROW5
- SW48 pad 1: /KeyMatrix/COL10 -> /KeyMatrix/COL6
Routing:
- net /KeyMatrix/COL6: track 82.6 -> 181.9 mm, vias 5 -> 7
- net /KeyMatrix/COL7: track 85.3 -> 162.8 mm
- net /KeyMatrix/COL8: track 113.5 -> 190.1 mm, vias 4 -> 6
- net /KeyMatrix/ROW2: track 169.3 -> 226.5 mm, vias 0 -> 2
- net /KeyMatrix/ROW5: track 76.4 -> 67.9 mm
Other:
- outline, holes or cut-outs redrawn
