File: DESIGN FILES/KeyMatrix.sch (KiCad schematic (older format))
At the start: 100 parts, among them SW10 CherryMX, SW11 CherryMX, SW12 CherryMX, SW13 CherryMX, SW14 CherryMX, SW15 CherryMX, SW16 CherryMX, SW17 CherryMX, SW18 CherryMX, SW19 CherryMX, SW2 CherryMX, SW20 CherryMX, SW21 CherryMX, SW22 CherryMX, SW23 CherryMX, SW24 CherryMX, SW25 CherryMX, SW26 CherryMX, SW27 CherryMX, SW28 CherryMX, SW29 CherryMX, SW3 CherryMX, SW30 CherryMX, SW31 CherryMX, SW32 CherryMX, SW33 CherryMX, SW34 CherryMX, SW35 CherryMX, SW36 CherryMX, SW37 CherryMX, SW38 CherryMX, SW39 CherryMX, SW4 CherryMX, SW40 CherryMX, SW41 CherryMX, SW42 CherryMX, SW43 CherryMX, SW44 CherryMX, SW45 CherryMX, SW46 CherryMX, SW47 CherryMX, SW48 CherryMX, SW49 CherryMX, SW5 CherryMX, SW50 CherryMX, SW51 CherryMX, SW6 CherryMX, SW7 CherryMX, SW8 CherryMX, SW9 CherryMX

Commit message: Added custom MV PNs to each component
Added unique MV PN for each unique component, referenced in personal component database.
Parts:
- D1, D10, D11, D12, D13, D14, D15, D16, D17, D18, D19, D2, D20, D21, D22, D23, D24, D25, D26, D27, D28, D29, D3, D30, D31, D32, D33, D34, D35, D36, D37, D38, D39, D4, D40, D41, D42, D43, D44, D45, D46, D47, D48, D49, D5, D50, D6, D7, D8, D9: MV PN (none) -> 20004-A
- SW10, SW11, SW12, SW13, SW14, SW15, SW16, SW17, SW18, SW19, SW2, SW20, SW21, SW22, SW23, SW24, SW25, SW26, SW27, SW28, SW29, SW3, SW30, SW31, SW32, SW33, SW34, SW35, SW36, SW37, SW38, SW39, SW4, SW40, SW41, SW42, SW43, SW44, SW45, SW46, SW47, SW48, SW49, SW5, SW50, SW51, SW6, SW7, SW8, SW9: MV PN (none) -> DNP
